File: new_middle_inner/new_middle_inner.kicad_pcb (KiCad board)
At the start: 2 copper layers, 58 x 58 mm, 3 parts, among them J104 Conn_01x01_Pin, J105 Conn_01x01_Pin, J106 Conn_01x01_Pin

Commit message: checkpoint
Parts:
- J104, J105, J106: moved to F.Cu
- turned J104 to 0 degrees
