File: new_middle/new_middle.kicad_pcb (KiCad board)
At the start: 2 copper layers, 98 x 98 mm, 6 parts, among them J101 Conn_01x01_Pin, J102 Conn_01x01_Pin, J103 Conn_01x01_Pin, J104 Conn_01x01_Pin, J105 Conn_01x01_Pin, J106 Conn_01x01_Pin

Commit message: checkpoint
Parts:
- J101, J102, J103, J104, J105, J106: moved to F.Cu
- turned J101 to 0 degrees
- turned J103 to 120 degrees
- turned J104 to 0 degrees

Commit message: checkpoint
Parts:
- removed J104, J105, J106: Conn_01x01_Pin, MyPinSocket:MyPinSocket
Other:
- outline, holes or cut-outs redrawn
Changed lines of the file:
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@@
   (net 2 "unconnected-(J102-Pin_1-Pad1)")
   (net 3 "unconnected-(J103-Pin_1-Pad1)")
-  (net 4 "unconnected-(J104-Pin_1-Pad1)")
-  (net 5 "unconnected-(J105-Pin_1-Pad1)")
-  (net 6 "unconnected-(J106-Pin_1-Pad1)")
-  (footprint "MyPinSocket:MyPinSocket" (layer "F.Cu")
-    (at 22.5 50)
-    (descr "Through hole straight socket strip, 1x01, 2.54mm pitch, single row (from Kicad 4.0.7), script generated")
-    (tags "Through hole socket strip THT 1x01 2.54mm single row")
-    (property "Sheetfile" "new_middle.kicad_sch")
-    (property "Sheetname" "")
-    (property "ki_description" "Generic connector, single row, 01x01, script generated")
-    (property "ki_keywords" "connector")
-    (attr through_hole)
-    (fp_text reference "J104" (at 0 -2.77) (layer "F.SilkS")
-        (effects (font (size 1 1) (thickness 0.15)))
-    )
-    (fp_text value "Conn_01x01_Pin" (at 0 2.77) (layer "F.Fab")
-        (effects (font (size 1 1) (thickness 0.15)))
-    )
-    (fp_text user "${REFERENCE}" (at 0 0) (layer "F.Fab")
-        (effects (font (size 1 1) (thickness 0.15)))
-    )
-    (fp_line (start -1.33 1.21) (end -1.33 1.33)
-      (stroke (width 0.12) (type solid)) (layer "F.SilkS"))
-    (fp_line (start -1.33 1.33) (end 1.33 1.33)
-      (stroke (width 0.12) (type solid)) (layer "F.SilkS"))
-    (fp_line (start 0 -1.33) (end 1.33 -1.33)
-      (stroke (width 0.12) (type solid)) (layer "F.SilkS"))
-    (fp_line (start 1.33 -1.33) (end 1.33 0)
-      (stroke (width 0.12) (type solid)) (layer "F.SilkS"))
-    (fp_line (start 1.33 1.21) (end 1.33 1.33)
-      (stroke (width 0.12) (type solid)) (layer "F.SilkS"))
-    (fp_line (start -1.27 -1.27) (end 0.635 -1.27)
-      (stroke (width 0.1) (type solid)) (layer "F.Fab"))
-    (fp_line (start -1.27 1.27) (end -1.27 -1.27)
-      (stroke (width 0.1) (type solid)) (layer "F.Fab"))
-    (fp_line (start 0.635 -1.27) (end 1.27 -0.635)
-      (stroke (width 0.1) (type solid)) (layer "F.Fab"))
-    (fp_line (start 1.27 -0.635) (end 1.27 1.27)
-      (stroke (width 0.1) (type solid)) (layer "F.Fab"))
-    (fp_line (start 1.27 1.27) (end -1.27 1.27)
-      (stroke (width 0.1) (type solid)) (layer "F.Fab"))
-    (pad "1" thru_hole rect (at 0 0) (size 1.7 1.7) (drill 1) (layers "*.Cu" "*.Mask")
-      (net 4 "unconnected-(J104-Pin_1-Pad1)") (pinfunction "Pin_1") (pintype "passive"))
-    (model "${KICAD6_3DMODEL_DIR}/Connector_PinSocket_2.54mm.3dshapes/PinSocket_1x01_P2.54mm_Vertical.wrl"
-      (offset (xyz 0 0 0))
-      (scale (xyz 1 1 1))
-      (rotate (xyz 0 0 0))
-    )
-  )
   (footprint "MyPinSocket:MyPinSocket" (layer "F.Cu")
     (at 65.75 22.72 60)
@@
     )
   )
-  (footprint "MyPinSocket:MyPinSocket" (layer "F.Cu")
-    (at 63.75 73.816 120)
-    (descr "Through hole straight socket strip, 1x01, 2.54mm pitch, single row (from Kicad 4.0.7), script generated")
-    (tags "Through hole socket strip THT 1x01 2.54mm single row")
-    (property "Sheetfile" "new_middle.kicad_sch")
-    (property "Sheetname" "")
-    (property "ki_description" "Generic connector, single row, 01x01, script generated")
-    (property "ki_keywords" "connector")
-    (attr through_hole)
-    (fp_text reference "J106" (at 0 -2.77 120) (layer "F.SilkS")
-        (effects (font (size 1 1) (thickness 0.15)))
-    )
-    (fp_text value "Conn_01x01_Pin" (at 0 2.77 120) (layer "F.Fab")
-        (effects (font (size 1 1) (thickness 0.15)))
-    )
-    (fp_text user "${REFERENCE}" (at 0 0 120) (layer "F.Fab")
-        (effects (font (size 1 1) (thickness 0.15)))
-    )
-    (fp_line (start -1.33 1.21) (end -1.33 1.33)
-      (stroke (width 0.12) (type solid)) (layer "F.SilkS"))
-    (fp_line (start -1.33 1.33) (end 1.33 1.33)
-      (stroke (width 0.12) (type solid)) (layer "F.SilkS"))
-    (fp_line (start 0 -1.33) (end 1.33 -1.33)
-      (stroke (width 0.12) (type solid)) (layer "F.SilkS"))
-    (fp_line (start 1.33 -1.33) (end 1.33 0)
-      (stroke (width 0.12) (type solid)) (layer "F.SilkS"))
-    (fp_line (start 1.33 1.21) (end 1.33 1.33)
-      (stroke (width 0.12) (type solid)) (layer "F.SilkS"))
-    (fp_line (start -1.27 -1.27) (end 0.635 -1.27)
-      (stroke (width 0.1) (type solid)) (layer "F.Fab"))
-    (fp_line (start -1.27 1.27) (end -1.27 -1.27)
-      (stroke (width 0.1) (type solid)) (layer "F.Fab"))
-    (fp_line (start 0.635 -1.27) (end 1.27 -0.635)
-      (stroke (width 0.1) (type solid)) (layer "F.Fab"))
-    (fp_line (start 1.27 -0.635) (end 1.27 1.27)
-      (stroke (width 0.1) (type solid)) (layer "F.Fab"))
-    (fp_line (start 1.27 1.27) (end -1.27 1.27)
-      (stroke (width 0.1) (type solid)) (layer "F.Fab"))
-    (pad "1" thru_hole rect (at 0 0 120) (size 1.7 1.7) (drill 1) (layers "*.Cu" "*.Mask")
-      (net 6 "unconnected-(J106-Pin_1-Pad1)") (pinfunction "Pin_1") (pintype "passive"))
-    (model "${KICAD6_3DMODEL_DIR}/Connector_PinSocket_2.54mm.3dshapes/PinSocket_1x01_P2.54mm_Vertical.wrl"
-      (offset (xyz 0 0 0))
-      (scale (xyz 1 1 1))
-      (rotate (xyz 0 0 0))
-    )
-  )
-  (footprint "MyPinSocket:MyPinSocket" (layer "F.Cu")
-    (at 63.75 26.184 60)
-    (descr "Through hole straight socket strip, 1x01, 2.54mm pitch, single row (from Kicad 4.0.7), script generated")
-    (tags "Through hole socket strip THT 1x01 2.54mm single row")
-    (property "Sheetfile" "new_middle.kicad_sch")
-    (property "Sheetname" "")
-    (property "ki_description" "Generic connector, single row, 01x01, script generated")
-    (property "ki_keywords" "connector")
-    (attr through_hole)
-    (fp_text reference "J105" (at 0 -2.77 60) (layer "F.SilkS")
-        (effects (font (size 1 1) (thickness 0.15)))
-    )
-    (fp_text value "Conn_01x01_Pin" (at 0 2.77 60) (layer "F.Fab")
-        (effects (font (size 1 1) (thickness 0.15)))
-    )
-    (fp_text user "${REFERENCE}" (at 0 0 60) (layer "F.Fab")
-        (effects (font (size 1 1) (thickness 0.15)))
-    )
-    (fp_line (start -1.33 1.21) (end -1.33 1.33)
-      (stroke (width 0.12) (type solid)) (layer "F.SilkS"))
-    (fp_line (start -1.33 1.33) (end 1.33 1.33)
-      (stroke (width 0.12) (type solid)) (layer "F.SilkS"))
-    (fp_line (start 0 -1.33) (end 1.33 -1.33)
-      (stroke (width 0.12) (type solid)) (layer "F.SilkS"))
-    (fp_line (start 1.33 -1.33) (end 1.33 0)
-      (stroke (width 0.12) (type solid)) (layer "F.SilkS"))
-    (fp_line (start 1.33 1.21) (end 1.33 1.33)
-      (stroke (width 0.12) (type solid)) (layer "F.SilkS"))
-    (fp_line (start -1.27 -1.27) (end 0.635 -1.27)
-      (stroke (width 0.1) (type solid)) (layer "F.Fab"))
-    (fp_line (start -1.27 1.27) (end -1.27 -1.27)
-      (stroke (width 0.1) (type solid)) (layer "F.Fab"))
-    (fp_line (start 0.635 -1.27) (end 1.27 -0.635)
-      (stroke (width 0.1) (type solid)) (layer "F.Fab"))
-    (fp_line (start 1.27 -0.635) (end 1.27 1.27)
-      (stroke (width 0.1) (type solid)) (layer "F.Fab"))
-    (fp_line (start 1.27 1.27) (end -1.27 1.27)
-      (stroke (width 0.1) (type solid)) (layer "F.Fab"))
-    (pad "1" thru_hole rect (at 0 0 60) (size 1.7 1.7) (drill 1) (layers "*.Cu" "*.Mask")
-      (net 5 "unconnected-(J105-Pin_1-Pad1)") (pinfunction "Pin_1") (pintype "passive"))
-    (model "${KICAD6_3DMODEL_DIR}/Connector_PinSocket_2.54mm.3dshapes/PinSocket_1x01_P2.54mm_Vertical.wrl"
-      (offset (xyz 0 0 0))
-      (scale (xyz 1 1 1))
-      (rotate (xyz 0 0 0))
-    )
-  )
-  (gr_circle (center 50 50) (end 67 50)
-    (stroke (width 1.2) (type default)) (fill none) (layer "B.Cu"))
-  (gr_circle (center 50 50) (end 65 50)
-    (stroke (width 1.2) (type default)) (fill none) (layer "B.Cu"))
   (gr_circle (center 50 50) (end 96 50)
     (stroke (width 1.2) (type default)) (fill none) (layer "B.Cu"))
@@
   (gr_line (start 18.5 50) (end 4.2 50)
     (stroke (width 1.6) (type default)) (layer "B.Cu"))
-  (gr_circle (center 50 50) (end 63 50)
-    (stroke (width 1.2) (type default)) (fill none) (layer "B.Cu"))
   (gr_line (start 65.75 77.28) (end 70.9 86.2)
     (stroke (width 1.6) (type default)) (layer "B.Cu"))
   (gr_circle (center 50 50) (end 92 50)
     (stroke (width 1.2) (type default)) (fill none) (layer "B.Cu"))
-  (gr_line (start 63.75 26.184) (end 57.6 36.836)
-    (stroke (width 1.6) (type default)) (layer "B.Cu"))
-  (gr_line (start 63.75 73.816) (end 56.6 61.432)
-    (stroke (width 1.6) (type default)) (layer "B.Cu"))
-  (gr_line (start 22.5 50) (end 32.8 50)
-    (stroke (width 1.6) (type default)) (layer "B.Cu"))
   (gr_circle (center 50 50) (end 99 50)
     (stroke (width 0.1) (type default)) (fill none) (layer "Edge.Cuts"))
   (gr_circle (center 50 50) (end 80 50)
     (stroke (width 0.1) (type default)) (fill none) (layer "Edge.Cuts"))
-  (gr_circle (center 50 50) (end 79 50)
-    (stroke (width 0.1) (type default)) (fill none) (layer "Edge.Cuts"))
 )
